Commit message: updated launch file

File: urdf/robot.urdf (robot description, URDF)
Before this commit: robot navvis, 5 links, 4 joints
Links:
- link laser_horiz: geometry collision cylinder length=.072 radius=.052; visual cylinder length=.072 radius=.052
- link laser_vert_bottom: geometry collision box size=0.062 0.062 0.087; visual box size=0.062 0.062 0.087
- link laser_vert_top_left: geometry collision box size=0.062 0.062 0.087; visual box size=0.062 0.062 0.087
- link laser_vert_top_right: geometry collision box size=0.062 0.062 0.087; visual box size=0.062 0.062 0.087

File: urdf/robot.xacro (robot description, xacro)
@@ -21,5 +21,5 @@
 	<xacro:laser name="laser_vert_top_right" parent="base" xyz ="0.2978 -0.1450 1.8451"  rpy ="-1.1760 0.6313 -1.9377"
 meshes="package://gazebo_plugins/test/multi_robot_scenario/meshes/laser" />
-	<xacro:laser name="laser_vert_left" parent="base"  xyz="0.2997 0.1531 01.8443"  rpy ="1.1780 0.6198 1.8560"
+	<xacro:laser name="laser_vert_top_left" parent="base"  xyz="0.2997 0.1531 01.8443"  rpy ="1.1780 0.6198 1.8560"
 meshes="package://gazebo_plugins/test/multi_robot_scenario/meshes/laser" />
 	<xacro:VLP-16 parent="base" name="laser_horiz" topic="laser_horiz/packets" hz="10"
